File: DesignLab.kicad_pcb (KiCad board)
At the start: 2 copper layers, 30 x 43 mm, 58 parts, among them J1 Conn_01x06_Male, J2 USB_B_Micro, J3 Conn_01x03_Male, J4 Conn_01x12, J5 Conn_01x02_Male, Q1 IRLML2060, Q2 IRLML6402, Q3 BC817, SW1 SW_Push, SW2 SW_Push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

Commit message: Layout PCB v0.2
almost finish layout pcb without error
Parts:
- moved TP8 2.97 mm to (217.9, 75.6)
- moved TP7 2.25 mm to (217.8, 72.8)
- moved TP6 1.19 mm to (218.0, 69.7)
- moved C3 0.41 mm to (195.9, 62.6)
Routing:
- net VCC: track 93.7 -> 137.8 mm, vias 1 -> 5
- net GND: track 2.19 -> 29.2 mm, vias 1 -> 19
- net Net-(D1-Pad3): track 5.32 -> 29.5 mm
- net /LCD_SDA: track 16.0 -> 23.9 mm
- net /PA12: track 20.7 -> 26.7 mm
- net /SWDIO: track 23.7 -> 29.2 mm
- net /PA11: track 15.9 -> 20.0 mm
- net /PA8: track 16.1 -> 16.7 mm
- added copper zone on B.Cu, net GND
- added copper zone on F.Cu, net GND
Other:
- board text added: "Design Lab 2022 Eit"
- board text added: "Made by:"
- board text added: "Mateusz Bik"
- board text added: "Mikołaj Markiel"
- board text added: "Piotr Mosurek"
